Commit message: adding grippers to finger joints

File: urdf/camera_mount.xacro (robot description, xacro)
@@ -8,12 +8,16 @@
       </visual>
       <collision>
+        <origin xyz="-0.0739 0 0.0245" rpy="0 0 0"/>
         <geometry>
-          <box size="0.12 0.06 0.065"/>
+          <box size="0.1178 0.060 0.0641"/>
         </geometry>
       </collision>
       <inertial>
+        <origin xyz="-0.0739 0 0.0245" rpy="0 0 0"/>
         <mass value="0.05"/>
-        <origin xyz="0 0 0" rpy="0 0 0"/>
-        <inertia ixx="1e-5" ixy="0" ixz="0" iyy="1e-5" iyz="0" izz="1e-5"/>
+        <inertia
+          ixx="${0.05/12*(0.060*0.060 + 0.0641*0.0641)}" ixy="0" ixz="0"
+          iyy="${0.05/12*(0.1178*0.1178 + 0.0641*0.0641)}" iyz="0"
+          izz="${0.05/12*(0.1178*0.1178 + 0.060*0.060)}"/>
       </inertial>
     </link>

File: urdf/prismatic_fr3_duo.urdf.xacro (robot description, xacro)
@@ -2,4 +2,6 @@
 <robot xmlns:xacro="http://www.ros.org/wiki/xacro" name="prismatic_fr3_duo">
   <xacro:include filename="./prismatic_fr3_duo.xacro"/>
+  <xacro:include filename="./camera_mount.xacro"/>
+  <xacro:include filename="./soft_gripper_finger.xacro"/>
   <xacro:arg name="config_file" default="../config/prismatic_fr3_duo.yaml"/>
   <xacro:property name="params" value="${xacro.load_yaml('$(arg config_file)')}"/>
@@ -27,3 +29,9 @@
     arm_prefixes="${params['arm_prefixes']}"
     no_prefix="${params['no_prefix']}"/>
+  <xacro:camera_mount prefix="left_" parent="left_fr3_hand"/>
+  <xacro:camera_mount prefix="right_" parent="right_fr3_hand"/>
+  <xacro:soft_gripper_finger suffix="left_fr3_leftfinger" parent="left_fr3_leftfinger"
+    xyz="0.0129 0 0.0362" rpy="3.1420 0 1.5521"/>
+  <xacro:soft_gripper_finger suffix="left_fr3_rightfinger" parent="left_fr3_rightfinger"
+    xyz="0.0129 0 0.0362" rpy="3.1420 0 1.5521"/>
 </robot>

File: urdf/prismatic_fr3_duo.xacro (robot description, xacro)
@@ -3,5 +3,4 @@
   <xacro:include filename="$(find franka_description)/robots/common/franka_robot.xacro"/>
   <xacro:include filename="./base_system.xacro"/>
-  <xacro:include filename="./camera_mount.xacro"/>
   <xacro:macro
     name="prismatic_fr3_duo"
@@ -33,5 +32,4 @@
         description_pkg="${description_pkg}"
         connected_to=""/>
-        <xacro:camera_mount prefix="${arm_prefix}" parent="${arm_prefix}${robot_type}_hand"/>
       <joint name="${arm_name}_base_joint" type="fixed">
         <parent link="base_link"/>

Commit message: changed d405 camera mount color to black

File: urdf/camera_mount.xacro (robot description, xacro)
@@ -6,4 +6,7 @@
           <mesh filename="package://prismatic_fr3_duo_description/meshes/d405_mount.stl" scale=".001 .001 .001"/>
         </geometry>
+        <material name="mount_black">
+          <color rgba="0.05 0.05 0.05 1"/>
+        </material>
       </visual>
       <collision>

Commit message: d405 added to urdf model

File: urdf/camera_mount.xacro (robot description, xacro)
@@ -30,4 +30,34 @@
       <origin xyz="0 0 0.008" rpy="0 0 0"/>
     </joint>
+    <link name="${prefix}d405">
+      <visual>
+        <origin xyz="-0.01 0 0.023" rpy="0 0 0"/>
+        <geometry>
+          <mesh filename="package://prismatic_fr3_duo_description/meshes/d405.stl" scale="1 1 1"/>
+        </geometry>
+        <material name="d405_original">
+          <color rgba="0.996078 0.996078 1 1"/>
+        </material>
+      </visual>
+      <collision>
+        <origin xyz="-0.01 0 0.0115" rpy="0 0 0"/>
+        <geometry>
+          <box size="0.042 0.042 0.023"/>
+        </geometry>
+      </collision>
+      <inertial>
+        <origin xyz="-0.01 0 0.0115" rpy="0 0 0"/>
+        <mass value="0.027"/>
+        <inertia
+          ixx="${0.027/12*(0.042*0.042 + 0.023*0.023)}" ixy="0" ixz="0"
+          iyy="${0.027/12*(0.042*0.042 + 0.023*0.023)}" iyz="0"
+          izz="${0.027/12*(0.042*0.042 + 0.042*0.042)}"/>
+      </inertial>
+    </link>
+    <joint name="${prefix}d405_joint" type="fixed">
+      <parent link="${prefix}camera_mount"/>
+      <child link="${prefix}d405"/>
+      <origin xyz="-0.125313 -0.0015 0.0360858" rpy="0.785398 0 1.5708"/>
+    </joint>
   </xacro:macro>
 </robot>

Commit message: fix: downpixeled stl

File: urdf/camera_mount.xacro (robot description, xacro)
@@ -34,5 +34,5 @@
         <origin xyz="-0.01 0 0.023" rpy="0 0 0"/>
         <geometry>
-          <mesh filename="package://prismatic_fr3_duo_description/meshes/d405.stl" scale="1 1 1"/>
+          <mesh filename="package://prismatic_fr3_duo_description/meshes/d405.stl" scale="0.001 0.001 0.001"/>
         </geometry>
         <material name="d405_original">

Commit message: fix:camera mount orientation, gripper mount addition

File: urdf/camera_mount.xacro (robot description, xacro)
@@ -11,5 +11,5 @@
       </visual>
       <collision>
-        <origin xyz="-0.0739 0 0.0245" rpy="0 0 0"/>
+        <origin xyz="-0.0739 0 0.0245" rpy="0 0 3.14150"/>
         <geometry>
           <box size="0.1178 0.060 0.0641"/>

File: urdf/soft_gripper_finger.xacro (robot description, xacro)
@@ -5,6 +5,6 @@
       <visual>
         <origin xyz="0.0129 0 0.0265134" rpy="3.1420 0 1.5708"/>
-        <geometry>
-          <mesh filename="package://prismatic_fr3_duo_description/meshes/soft_gripper_finger.stl" scale="0.001 0.001 0.001"/>
+          <geometry>
+          <mesh filename="package://prismatic_fr3_duo_description/meshes/mount+gripper.stl" scale="0.001 0.001 0.001"/>
         </geometry>
       </visual>

Commit message: fix: cameras revert direction and tcp for soft gripper

File: urdf/camera_mount.xacro (robot description, xacro)
@@ -28,5 +28,5 @@
       <parent link="${parent}"/>
       <child link="${prefix}camera_mount"/>
-      <origin xyz="0 0 0.008" rpy="0 0 0"/>
+      <origin xyz="0 0 0.008" rpy="0 0 ${pi}"/>
     </joint>
     <link name="${prefix}d405">

File: urdf/prismatic_fr3_duo.urdf (robot description, URDF)
Before this commit: robot prismatic_fr3_duo, 52 links, 51 joints
Links:
- added link left_camera_mount, mass 0.05; collision box size=0.1178 0.060 0.0641; visual mesh filename=package://prismatic_fr3_duo_description/meshes/d405_mount.s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 scale=.001 .001 .001
- added link left_d405, mass 0.027; collision box size=0.042 0.042 0.023; visual mesh filename=package://prismatic_fr3_duo_description/meshes/d405.stl scale=0.001 0.001 0.001
- added link left_fr3_leftfinger_soft_finger, mass 0.02; collision box size=0.040 0.04 .1234; visual mesh filename=package://prismatic_fr3_duo_description/meshes/mount_grippe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 scale=0.001 0.001 0.001
- added link left_fr3_rightfinger_soft_finger, mass 0.02; collision box size=0.040 0.04 .1234; visual mesh filename=package://prismatic_fr3_duo_description/meshes/mount_grippe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 scale=0.001 0.001 0.001
- added link right_camera_mount, mass 0.05; collision box size=0.1178 0.060 0.0641; visual mesh filename=package://prismatic_fr3_duo_description/meshes/d405_mount.s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 scale=.001 .001 .001
- added link right_d405, mass 0.027; collision box size=0.042 0.042 0.023; visual mesh filename=package://prismatic_fr3_duo_description/meshes/d405.stl scale=0.001 0.001 0.001
- added link right_fr3_leftfinger_soft_finger, mass 0.02; collision box size=0.040 0.04 .1234; visual mesh filename=package://prismatic_fr3_duo_description/meshes/mount_grippe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 scale=0.001 0.001 0.001
- added link right_fr3_rightfinger_soft_finger, mass 0.02; collision box size=0.040 0.04 .1234; visual mesh filename=package://prismatic_fr3_duo_description/meshes/mount_grippe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 scale=0.001 0.001 0.001
- link left_fr3_hand: geometry collision mesh filename=package://franka_description/meshes/robot_ee/franka_hand_wh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; visual mesh filename=package://franka_description/meshes/robot_ee/franka_hand_wh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
- link left_fr3_leftfinger: geometry collision box size=17.5e-3 15.2e-3 18.5e-3; collision box size=17.5e-3 7e-3 23.5e-3
- link left_fr3_link0: geometry collision mesh filename=package://franka_description/meshes/robots/fr3/collision/li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; visual mesh filename=package://franka_description/meshes/robots/fr3/visual/link0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
- link left_fr3_link1: geometry collision mesh filename=package://franka_description/meshes/robots/fr3/collision/li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; visual mesh filename=package://franka_description/meshes/robots/fr3/visual/link1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
- link left_fr3_link2: geometry collision mesh filename=package://franka_description/meshes/robots/fr3/collision/li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; visual mesh filename=package://franka_description/meshes/robots/fr3/visual/link2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
- link left_fr3_link3: geometry collision mesh filename=package://franka_description/meshes/robots/fr3/collision/li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; visual mesh filename=package://franka_description/meshes/robots/fr3/visual/link3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
- link left_fr3_link4: geometry collision mesh filename=package://franka_description/meshes/robots/fr3/collision/li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; visual mesh filename=package://franka_description/meshes/robots/fr3/visual/link4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
- link left_fr3_link5: geometry collision mesh filename=package://franka_description/meshes/robots/fr3/collision/li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; visual mesh filename=package://franka_description/meshes/robots/fr3/visual/link5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
- link left_fr3_link6: geometry collision mesh filename=package://franka_description/meshes/robots/fr3/collision/li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; visual mesh filename=package://franka_description/meshes/robots/fr3/visual/link6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
- link left_fr3_link7: geometry collision mesh filename=package://franka_description/meshes/robots/fr3/collision/li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; visual mesh filename=package://franka_description/meshes/robots/fr3/visual/link7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
- link left_fr3_rightfinger: geometry collision box size=17.5e-3 15.2e-3 18.5e-3; collision box size=17.5e-3 7e-3 23.5e-3
- link right_fr3_hand: geometry collision mesh filename=package://franka_description/meshes/robot_ee/franka_hand_wh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; visual mesh filename=package://franka_description/meshes/robot_ee/franka_hand_wh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
- link right_fr3_leftfinger: geometry collision box size=17.5e-3 15.2e-3 18.5e-3; collision box size=17.5e-3 7e-3 23.5e-3
- link right_fr3_link0: geometry collision mesh filename=package://franka_description/meshes/robots/fr3/collision/li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; visual mesh filename=package://franka_description/meshes/robots/fr3/visual/link0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
- link right_fr3_link1: geometry collision mesh filename=package://franka_description/meshes/robots/fr3/collision/li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; visual mesh filename=package://franka_description/meshes/robots/fr3/visual/link1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
- link right_fr3_link2: geometry collision mesh filename=package://franka_description/meshes/robots/fr3/collision/li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; visual mesh filename=package://franka_description/meshes/robots/fr3/visual/link2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
- link right_fr3_link3: geometry collision mesh filename=package://franka_description/meshes/robots/fr3/collision/li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; visual mesh filename=package://franka_description/meshes/robots/fr3/visual/link3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
- link right_fr3_link4: geometry collision mesh filename=package://franka_description/meshes/robots/fr3/collision/li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; visual mesh filename=package://franka_description/meshes/robots/fr3/visual/link4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
- link right_fr3_link5: geometry collision mesh filename=package://franka_description/meshes/robots/fr3/collision/li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; visual mesh filename=package://franka_description/meshes/robots/fr3/visual/link5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
- link right_fr3_link6: geometry collision mesh filename=package://franka_description/meshes/robots/fr3/collision/li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; visual mesh filename=package://franka_description/meshes/robots/fr3/visual/link6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
- link right_fr3_link7: geometry collision mesh filename=package://franka_description/meshes/robots/fr3/collision/li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; visual mesh filename=package://franka_description/meshes/robots/fr3/visual/link7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
- link right_fr3_rightfinger: geometry collision box size=17.5e-3 15.2e-3 18.5e-3; collision box size=17.5e-3 7e-3 23.5e-3
Joints:
- added joint left_camera_mount_joint: type fixed, parent left_fr3_hand, child left_camera_mount, origin xyz=0 0 0.008 rpy=0 0 3.141592653589793
- added joint left_d405_joint: type fixed, parent left_camera_mount, child left_d405, origin xyz=-0.125313 -0.0015 0.0360858 rpy=0.785398 0 1.5708
- added joint left_fr3_leftfinger_soft_finger_joint: type fixed, parent left_fr3_leftfinger, child left_fr3_leftfinger_soft_finger, origin xyz=0 0 0 rpy=0 0 0
- added joint left_fr3_rightfinger_soft_finger_joint: type fixed, parent left_fr3_rightfinger, child left_fr3_rightfinger_soft_finger, origin xyz=0 0 0 rpy=0 0 0
- added joint right_camera_mount_joint: type fixed, parent right_fr3_hand, child right_camera_mount, origin xyz=0 0 0.008 rpy=0 0 3.141592653589793
- added joint right_d405_joint: type fixed, parent right_camera_mount, child right_d405, origin xyz=-0.125313 -0.0015 0.0360858 rpy=0.785398 0 1.5708
- added joint right_fr3_leftfinger_soft_finger_joint: type fixed, parent right_fr3_leftfinger, child right_fr3_leftfinger_soft_finger, origin xyz=0 0 0 rpy=0 0 0
- added joint right_fr3_rightfinger_soft_finger_joint: type fixed, parent right_fr3_rightfinger, child right_fr3_rightfinger_soft_finger, origin xyz=0 0 0 rpy=0 0 0
- joint left_fr3_hand_tcp_joint: origin xyz=0 0 0.1034 rpy=0 0 1.5707963267948966 -> xyz=0 0 0.195 rpy=0 0 1.5707963267948966
- joint right_fr3_hand_tcp_joint: origin xyz=0 0 0.1034 rpy=0 0 1.5707963267948966 -> xyz=0 0 0.195 rpy=0 0 1.5707963267948966

File: urdf/soft_gripper_finger.xacro (robot description, xacro)
@@ -6,5 +6,5 @@
         <origin xyz="0.0129 0 0.0265134" rpy="3.1420 0 1.5708"/>
           <geometry>
-          <mesh filename="package://prismatic_fr3_duo_description/meshes/mount+gripper.stl" scale="0.001 0.001 0.001"/>
+          <mesh filename="package://prismatic_fr3_duo_description/meshes/mount_gripper.stl" scale="0.001 0.001 0.001"/>
         </geometry>
       </visual>
